Commit message: ホイールオドメトリを有効化

File: xacro/gunrobo.xacro (robot description, xacro)
@@ -10,5 +10,5 @@
     <xacro:property name="wheel_w_size" value="0.02" />
     <xacro:property name="wheel_y_shift" value="0.03" />
-    <xacro:property name="ball_size" value="0.005" />
+    <xacro:property name="ball_size" value="0.0048" />
     <xacro:property name="ball_shift" value="0.1" />
     <link name="base_footprint" >
@@ -69,10 +69,4 @@
             <legacyModeNS>true</legacyModeNS>
         </plugin>
-        <plugin name="ground_truth" filename="libgazebo_ros_p3d.so">
-            <frameName>map</frameName>
-            <bodyName>base_footprint</bodyName>
-            <topicName>/tracker</topicName>
-            <updateRate>10.0</updateRate>
-        </plugin>
     </gazebo>
 </robot>

File: xacro/wheel.xacro (robot description, xacro)
@@ -49,6 +49,6 @@
         <gazebo reference="${wheel_link}">
             <material>Gazebo/Red</material>
-            <mu1>0.05</mu1>
-            <mu2>0.05</mu2>
+            <mu1>0.75</mu1>
+            <mu2>0.75</mu2>
         </gazebo>
     </xacro:macro>

Commit message: ちゃんと動くようにパラメータを調整
- 滑っている原因は、massもしくはinnertiaの設定値が小さすぎたため
- wheelがガタガタ振動していたのも、上記と同じ修正になった

File: xacro/gunrobo.xacro (robot description, xacro)
@@ -31,5 +31,5 @@
         </visual>
         <inertial>
-            <xacro:property name="mass" value="0.1" />
+            <xacro:property name="mass" value="20" />
             <xacro:property name="inertia_sphere" value="${mass*w_size*w_size/5}" />
             <mass value="${mass}"/>
@@ -46,5 +46,5 @@
         <origin
             xyz="0.0 ${w_size / 2 + wheel_y_shift} ${- w_size / 2 + wheel_r_size - lift_up}"
-            rpy="${pi/2} 0.0 0.0" />
+            rpy="${-pi/2} 0.0 0.0" />
         <axis xyz="0.0 0.0 1.0" />
     </xacro:wheel>

File: xacro/wheel.xacro (robot description, xacro)
@@ -29,5 +29,5 @@
             </collision>
             <inertial>
-                <xacro:property name="mass" value="0.1" />
+                <xacro:property name="mass" value="1" />
                 <xacro:property name="inertia_ixx" value="${mass*r_size*r_size/4 + mass*w_size*w_size/12}" />
                 <xacro:property name="inertia_izz" value="${mass*r_size*r_size/2}" />
@@ -49,6 +49,6 @@
         <gazebo reference="${wheel_link}">
             <material>Gazebo/Red</material>
-            <mu1>0.75</mu1>
-            <mu2>0.75</mu2>
+            <mu1>0.9</mu1>
+            <mu2>0.9</mu2>
         </gazebo>
     </xacro:macro>
